File: Electrical Design/PCB/PCB.sch (KiCad schematic (older format))
At the start: 19 parts

Commit message: Added SS490 Hall effect symbol
Parts:
- added U?: SS490_Hall_Sensor, symbol Custom_Components:SS490_Hall_Sensor
Connections:
- wire segments 49 -> 51
Changed lines of the file:
@@
 	1    0    0    -1
 $EndComp
+$Comp
+L Custom_Components:SS490_Hall_Sensor U?
+U 1 1 5C2E0303
+P 3300 1750
+F 0 "U?" H 3481 2525 50  0000 C CNN
+F 1 "SS490_Hall_Sensor" H 3481 2434 50  0000 C CNN
+F 2 "" H 3400 2650 50  0001 C CNN
+F 3 "" H 3400 2650 50  0001 C CNN
+	1    3300 1750
+	1    0    0    -1
+$EndComp
+$Comp
+L power:GND #PWR?
+U 1 1 5C2E0666
+P 3750 1450
+F 0 "#PWR?" H 3750 1200 50  0001 C CNN
+F 1 "GND" H 3755 1277 50  0000 C CNN
+F 2 "" H 3750 1450 50  0001 C CNN
+F 3 "" H 3750 1450 50  0001 C CNN
+	1    3750 1450
+	1    0    0    -1
+$EndComp
+Wire Wire Line
+	3750 1450 3750 1400
+Wire Wire Line
+	3750 1400 3650 1400
 $EndSCHEMATC

Commit message: Electrical Overhaul
Parts:
- removed C? (x2): 100nF, symbol Device:C
- removed C? (x2): 10μF, symbol Device:CP1
- removed C?: 100nF, symbol Device:C_Small
- removed C? (x3): 22µF, symbol Device:C_Small
- removed C?: 22pF, symbol Device:C_Small
- removed FB?: Ferrite_Bead_Small, symbol Device:Ferrite_Bead_Small
- removed J?: Header 3x2, symbol Connector_Generic:Conn_02x03_Odd_Even
- removed L?: 10μH, symbol pspice:INDUCTOR
- removed L?: 2.2µH, symbol Device:L_Small
- removed R?: 10kΩ, symbol Device:R_Small
- removed R?: 150kΩ, symbol Device:R_Small
- removed R?: 300kΩ, symbol Device:R_Small
- removed U?: ATxmega128A1U-AU, Package_QFP:TQFP-100_14x14mm_P0.5mm, symbol MCU_Microchip_ATmega:ATxmega128A1U-AU
- removed U?: MS5607, symbol Custom_Components:MS5607
- removed U?: AP3419, symbol Custom_Components:AP3419
- removed U?: SS490_Hall_Sensor, symbol Custom_Components:SS490_Hall_Sensor
- added C? (x2): 10uF, symbol Device:CP1_Small
- added C? (x3): 100nF, symbol Device:C_Small
- added C? (x3): 0.1uF, symbol Device:CP1_Small
- added C? (x2): 22pF, symbol Device:CP1_Small
- added C? (x5): 1uF, symbol Device:C_Small
- added FB?: 220@100MHz, symbol Device:Ferrite_Bead_Small
- added J?: Conn_02x03_Odd_Even, symbol Connector_Generic:Conn_02x03_Odd_Even
- added L?: 10uH, symbol Device:L_Small
- added R?: 10k, symbol Device:R_Small
- added R?: R_Small, symbol Device:R_Small
- added TH?: NTCLE100, symbol Device:Thermistor_NTC
- added U?: ATxmega128A4U-AU, Package_QFP:TQFP-44_10x10mm_P0.8mm, symbol MCU_Microchip_ATmega:ATxmega128A4U-AU
- added U?: MS560702BA03-50, SON125P300X500X100-8N, symbol MS560702BA03-50:MS560702BA03-50
- added U?: BNO080, LGA-28, symbol BNO080:BNO080
- added U?: ADP3338AKCZ-5-R7, SOT230P700X180-4N, symbol ADP3338AKCZ-5-R7:ADP3338AKCZ-5-R7
- added U?: ADP3338AKCZ-3.3-R7, SOT230P700X180-4N, symbol ADP3338AKCZ-5-R7:ADP3338AKCZ-5-R7
- added U?: SS495A, SIP3-UA, symbol SS495A:SS495A
- added Y?: ?, symbol Device:Crystal
Connections:
- net labels added: -3V3, -5V, ADC, BNO_BOOTN, BNO_CLOCKSEL0, BNO_NRST, BNO_WAKE, ENV_SCL, ENV_SDA, HOST_CSN, HOST_INTN, MCU_AVCC, MCU_VCC, PDI_CLK, PDI_DATA, SCLK, SDI, SDO, UNASSIGNED, VCC
- wire segments 51 -> 97
- no-connect marks 0 -> 2

Commit message: m
Connections:
- net HOST_CSN is gone; now on net SS_BNO080: U?.18 (~H_CS~)
- net SDI is gone; now on net MOSI: U?.17 (H_SA0/MOSI), U?.7 (SDI/SDA)
- net SDO is gone; now on net MISO: U?.20 (H_SDA/MISO/TX), U?.6 (SDO)
- net SCLK: now also U?.17 (PC7)
- net UNASSIGNED: no longer U?.4 (~CSB~), U?.5 (~CSB~)
- net SS_BNO080: now reaches U?.13 (PC3)
- net SS_5607: now reaches U?.14 (PC4)
- net SS_5607: now also U?.4 (~CSB~), U?.5 (~CSB~)
- net MOSI: now reaches U?.15 (PC5)
- net MISO: now reaches U?.16 (PC6)
- net RX: now reaches U?.22 (PD2)
- net TX: now reaches U?.23 (PD3)
- net TC: now reaches U?.24 (PD4)
- net TC: now also U?.25 (PD5)
Other:
- note added: "Ports A & B have access to the ADC"
- moved on the sheet: C?, FB?, J?, L?, R?, TH?, U?

Commit message: uodate
Parts:
- added R?: 10, symbol Device:R_Small
- added R?: 5, symbol Device:R_Small
Connections:
- net +3V3: now also R?.2
- net GND: now also R?.1
- net PA7-Voltage: now reaches U?.3 (PA7)
- net PA7-Voltage: now also R?.1, R?.2
- net ENV_SCL: no longer names the net of U?.15 (S_SCL)
- net ENV_SDA: no longer names the net of U?.16 (S_SDA)
- no-connect marks 2 -> 4
Other:
- note added: "6V —> 3.3V Regulator"
- note added: "6V —> 5V Regulator"
- note added: "BNO-080"
- note added: "Hall Effect Sensor"
- note added: "MS5607 Pressure Sensor"
- note added: "PDI Interface"
- note added: "Power Interface"
- note added: "Thermistor"
- note added: "Voltage Divider (3.3 —> 2.2)"
- moved on the sheet: J?, R?
Changed lines of the file:
@@
 L Connector_Generic:Conn_02x03_Odd_Even J?
 U 1 1 5C487514
-P 1550 4200
-F 0 "J?" H 1600 4500 50  0000 C CNN
-F 1 "Conn_02x03_Odd_Even" H 1600 4400 50  0000 C CNN
-F 2 "" H 1550 4200 50  0001 C CNN
-F 3 "~" H 1550 4200 50  0001 C CNN
-	1    1550 4200
-	1    0    0    -1
-$EndComp
-NoConn ~ 1850 4200
-NoConn ~ 1350 4200
+P 1150 4250
+F 0 "J?" H 1200 4550 50  0000 C CNN
+F 1 "Conn_02x03_Odd_Even" H 1200 4450 50  0000 C CNN
+F 2 "" H 1150 4250 50  0001 C CNN
+F 3 "~" H 1150 4250 50  0001 C CNN
+	1    1150 4250
+	1    0    0    -1
+$EndComp
+NoConn ~ 1450 4250
+NoConn ~ 950  4250
 Text Label 7400 5750 0    50   ~ 0
 MCU_VCC
@@
 Text Label 7700 5650 0    50   ~ 0
 MCU_AVCC
-Text Label 1350 4100 2    50   ~ 0
+Text Label 950  4150 2    50   ~ 0
 PDI_DATA
 Text Label 8950 3650 2    50   ~ 0
@@
 L Device:R_Small R?
 U 1 1 5C48AF52
-P 2100 4300
-F 0 "R?" H 2159 4346 50  0000 L CNN
-F 1 "10k" H 2159 4255 50  0000 L CNN
-F 2 "" H 2100 4300 50  0001 C CNN
-F 3 "~" H 2100 4300 50  0001 C CNN
-	1    2100 4300
+P 1700 4350
+F 0 "R?" H 1759 4396 50  0000 L CNN
+F 1 "10k" H 1759 4305 50  0000 L CNN
+F 2 "" H 1700 4350 50  0001 C CNN
+F 3 "~" H 1700 4350 50  0001 C CNN
+	1    1700 4350
 	1    0    0    -1
 $EndComp
@@
 L power:GND #PWR0105
 U 1 1 5C48B786
-P 1850 4300
-F 0 "#PWR0105" H 1850 4050 50  0001 C CNN
-F 1 "GND" H 1855 4127 50  0000 C CNN
-F 2 "" H 1850 4300 50  0001 C CNN
-F 3 "" H 1850 4300 50  0001 C CNN
-	1    1850 4300
+P 1450 4350
+F 0 "#PWR0105" H 1450 4100 50  0001 C CNN
+F 1 "GND" H 1455 4177 50  0000 C CNN
+F 2 "" H 1450 4350 50  0001 C CNN
+F 3 "" H 1450 4350 50  0001 C CNN
+	1    1450 4350
 	1    0    0    -1
 $EndComp
@@
 L power:VDD #PWR0106
 U 1 1 5C48BD0F
-P 2100 3950
-F 0 "#PWR0106" H 2100 3800 50  0001 C CNN
-F 1 "VDD" H 2117 4123 50  0000 C CNN
-F 2 "" H 2100 3950 50  0001 C CNN
-F 3 "" H 2100 3950 50  0001 C CNN
-	1    2100 3950
-	1    0    0    -1
-$EndComp
-Wire Wire Line
-	1850 4100 2100 4100
-Wire Wire Line
-	2100 4100 2100 3950
-Connection ~ 2100 4100
-Wire Wire Line
-	2100 4100 2100 4200
-Wire Wire Line
-	1350 4300 1250 4300
-Wire Wire Line
-	1250 4300 1250 4500
-Wire Wire Line
-	1250 4500 2100 4500
-Wire Wire Line
-	2100 4500 2100 4400
+P 1700 4000
+F 0 "#PWR0106" H 1700 3850 50  0001 C CNN
+F 1 "VDD" H 1717 4173 50  0000 C CNN
+F 2 "" H 1700 4000 50  0001 C CNN
+F 3 "" H 1700 4000 50  0001 C CNN
+	1    1700 4000
+	1    0    0    -1
+$EndComp
+Wire Wire Line
+	1450 4150 1700 4150
+Wire Wire Line
+	1700 4150 1700 4000
+Connection ~ 1700 4150
+Wire Wire Line
+	1700 4150 1700 4250
+Wire Wire Line
+	950  4350 850  4350
+Wire Wire Line
+	850  4350 850  4550
+Wire Wire Line
+	850  4550 1700 4550
+Wire Wire Line
+	1700 4550 1700 4450
 Text Label 8950 3550 2    50   ~ 0
 PDI_CLK
-Text Label 2100 4550 3    50   ~ 0
+Text Label 1700 4600 3    50   ~ 0
 PDI_CLK
 $Comp
@@
 Text Label 2650 1400 0    50   ~ 0
 BNO_NRST
-Text Label 2650 1800 0    50   ~ 0
-ENV_SDA
-Text Label 2650 1900 0    50   ~ 0
-ENV_SCL
 $Comp
 L power:GND #PWR0113
@@
 SCLK
 Wire Wire Line
-	2100 4500 2100 4550
-Connection ~ 2100 4500
+	1700 4550 1700 4600
+Connection ~ 1700 4550
 Text Label 10350 5250 0    50   ~ 0
 SS_BNO080
@@
 Text GLabel 8950 5450 0    50   Input ~ 0
 TC
+NoConn ~ 2650 1800
+NoConn ~ 2650 1900
+$Comp
+L power:+3.3V #PWR?
+U 1 1 5C491155
+P 2200 4200
+F 0 "#PWR?" H 2200 4050 50  0001 C CNN
+F 1 "+3.3V" H 2215 4373 50  0000 C CNN
+F 2 "" H 2200 4200 50  0001 C CNN
+F 3 "" H 2200 4200 50  0001 C CNN
+	1    2200 4200
+	1    0    0    -1
+$EndComp
+$Comp
+L Device:R_Small R?
+U 1 1 5C491A8E
+P 2900 4300
+F 0 "R?" V 2704 4300 50  0000 C CNN
+F 1 "10" V 2795 4300 50  0000 C CNN
+F 2 "" H 2900 4300 50  0001 C CNN
+F 3 "~" H 2900 4300 50  0001 C CNN
+	1    2900 4300
+	0    1    1    0
+$EndComp
+$Comp
+L Device:R_Small R?
+U 1 1 5C491D93
+P 2500 4300
+F 0 "R?" V 2304 4300 50  0000 C CNN
+F 1 "5" V 2395 4300 50  0000 C CNN
+F 2 "" H 2500 4300 50  0001 C CNN
+F 3 "~" H 2500 4300 50  0001 C CNN
+	1    2500 4300
+	0    1    1    0
+$EndComp
+$Comp
+L power:GND #PWR?
+U 1 1 5C4998EE
+P 3200 4300
+F 0 "#PWR?" H 3200 4050 50  0001 C CNN
+F 1 "GND" V 3205 4172 50  0000 R CNN
+F 2 "" H 3200 4300 50  0001 C CNN
+F 3 "" H 3200 4300 50  0001 C CNN
+	1    3200 4300
+	0    -1   -1   0
+$EndComp
+Wire Wire Line
+	2200 4200 2200 4300
+Wire Wire Line
+	2200 4300 2400 4300
+Wire Wire Line
+	2600 4300 2700 4300
+Wire Wire Line
+	3000 4300 3200 4300
+Wire Wire Line
+	2700 4300 2700 4100
+Connection ~ 2700 4300
+Wire Wire Line
+	2700 4300 2800 4300
+Text Notes 2200 4500 0    50   ~ 0
+Voltage Divider (3.3 —> 2.2)
+Text Label 10350 4250 0    50   ~ 0
+PA7-Voltage
+Text Label 2700 4100 1    50   ~ 0
+PA7-Voltage
+Text Notes 4250 5100 0    50   ~ 0
+MS5607 Pressure Sensor
+Text Notes 6950 4950 0    50   ~ 0
+Power Interface
+Text Notes 5400 6650 0    50   ~ 0
+Hall Effect Sensor
+Text Notes 3050 6450 0    50   ~ 0
+6V —> 3.3V Regulator
+Text Notes 1350 5200 0    50   ~ 0
+6V —> 5V Regulator
+Text Notes 950  3800 0    50   ~ 0
+PDI Interface
+Text Notes 1700 3050 0    50   ~ 0
+BNO-080
+Text Notes 1200 6600 0    50   ~ 0
+Thermistor
 $EndSCHEMATC

Commit message: Add voltages
Connections:
- net ADC is gone; now on net PA6-Therm: R?.2, TH?.1
- net +3V3: now also C?.1, TH?.2, U?.1 (VDD)
- net VDD: no longer C?.1, C?.2, C?.2, TH?.2, U?.1 (VDD), U?.3 (IN), U?.3 (IN)
- net PA6-Therm: now reaches U?.2 (PA6)
- net VCC renamed +5V
- new net +6V: C?.2, C?.2, U?.3 (IN), U?.3 (IN)
Changed lines of the file:
@@
 Text Label 4150 5750 2    50   ~ 0
 SCLK
-$Comp
-L power:VDD #PWR0107
-U 1 1 5C48FB82
-P 5600 5450
-F 0 "#PWR0107" H 5600 5300 50  0001 C CNN
-F 1 "VDD" H 5617 5623 50  0000 C CNN
-F 2 "" H 5600 5450 50  0001 C CNN
-F 3 "" H 5600 5450 50  0001 C CNN
-	1    5600 5450
-	1    0    0    -1
-$EndComp
 Wire Wire Line
 	5350 5550 5600 5550
@@
 $EndComp
 $Comp
-L power:VDD #PWR0114
-U 1 1 5C4C9BA3
-P 750 6950
-F 0 "#PWR0114" H 750 6800 50  0001 C CNN
-F 1 "VDD" H 767 7123 50  0000 C CNN
-F 2 "" H 750 6950 50  0001 C CNN
-F 3 "" H 750 6950 50  0001 C CNN
-	1    750  6950
-	1    0    0    -1
-$EndComp
-$Comp
 L power:GND #PWR0115
 U 1 1 5C4C9DEF
@@
 	1250 6950 1400 6950
 Text Label 1400 7050 3    50   ~ 0
-ADC
+PA6-Therm
 $Comp
 L ADP3338AKCZ-5-R7:ADP3338AKCZ-5-R7 U?
@@
 $EndComp
 $Comp
-L power:VDD #PWR0116
-U 1 1 5C4D7B60
-P 700 5500
-F 0 "#PWR0116" H 700 5350 50  0001 C CNN
-F 1 "VDD" H 717 5673 50  0000 C CNN
-F 2 "" H 700 5500 50  0001 C CNN
-F 3 "" H 700 5500 50  0001 C CNN
-	1    700  5500
-	1    0    0    -1
-$EndComp
-$Comp
 L power:GND #PWR0117
 U 1 1 5C4D7F6B
@@
 $EndComp
 $Comp
-L power:VDD #PWR0121
-U 1 1 5C4ECC2A
-P 2400 6700
-F 0 "#PWR0121" H 2400 6550 50  0001 C CNN
-F 1 "VDD" H 2417 6873 50  0000 C CNN
-F 2 "" H 2400 6700 50  0001 C CNN
-F 3 "" H 2400 6700 50  0001 C CNN
-	1    2400 6700
-	1    0    0    -1
-$EndComp
-$Comp
 L power:GND #PWR0122
 U 1 1 5C4ECC30
@@
 F 8 "TO-92 Honeywell" H 5450 6900 50  0001 L BNN "Field8"
 	1    5450 6900
-	1    0    0    -1
-$EndComp
-$Comp
-L power:VCC #PWR0126
-U 1 1 5C4FE341
-P 5000 6950
-F 0 "#PWR0126" H 5000 6800 50  0001 C CNN
-F 1 "VCC" H 5017 7123 50  0000 C CNN
-F 2 "" H 5000 6950 50  0001 C CNN
-F 3 "" H 5000 6950 50  0001 C CNN
-	1    5000 6950
 	1    0    0    -1
 $EndComp
@@
 Text Notes 1200 6600 0    50   ~ 0
 Thermistor
+$Comp
+L power:+6V #PWR?
+U 1 1 5C49358D
+P 700 5500
+F 0 "#PWR?" H 700 5350 50  0001 C CNN
+F 1 "+6V" H 715 5673 50  0000 C CNN
+F 2 "" H 700 5500 50  0001 C CNN
+F 3 "" H 700 5500 50  0001 C CNN
+	1    700  5500
+	1    0    0    -1
+$EndComp
+$Comp
+L power:+6V #PWR?
+U 1 1 5C49758F
+P 2400 6700
+F 0 "#PWR?" H 2400 6550 50  0001 C CNN
+F 1 "+6V" H 2415 6873 50  0000 C CNN
+F 2 "" H 2400 6700 50  0001 C CNN
+F 3 "" H 2400 6700 50  0001 C CNN
+	1    2400 6700
+	1    0    0    -1
+$EndComp
+$Comp
+L power:+3.3V #PWR?
+U 1 1 5C49ACEC
+P 5600 5450
+F 0 "#PWR?" H 5600 5300 50  0001 C CNN
+F 1 "+3.3V" H 5615 5623 50  0000 C CNN
+F 2 "" H 5600 5450 50  0001 C CNN
+F 3 "" H 5600 5450 50  0001 C CNN
+	1    5600 5450
+	1    0    0    -1
+$EndComp
+$Comp
+L power:+3.3V #PWR?
+U 1 1 5C49E3CA
+P 750 6950
+F 0 "#PWR?" H 750 6800 50  0001 C CNN
+F 1 "+3.3V" H 765 7123 50  0000 C CNN
+F 2 "" H 750 6950 50  0001 C CNN
+F 3 "" H 750 6950 50  0001 C CNN
+	1    750  6950
+	1    0    0    -1
+$EndComp
+$Comp
+L power:+5V #PWR?
+U 1 1 5C4A1F82
+P 5000 6950
+F 0 "#PWR?" H 5000 6800 50  0001 C CNN
+F 1 "+5V" H 5015 7123 50  0000 C CNN
+F 2 "" H 5000 6950 50  0001 C CNN
+F 3 "" H 5000 6950 50  0001 C CNN
+	1    5000 6950
+	1    0    0    -1
+$EndComp
+Text Label 10350 4150 0    50   ~ 0
+PA6-Therm
 $EndSCHEMATC

Commit message: m
Connections:
- net VDD is gone; now on net +3V3: J?.2 (Pin_2), R?.1
Changed lines of the file:
@@
-	1    0    0    -1
-$EndComp
-$Comp
-L power:VDD #PWR0106
-U 1 1 5C48BD0F
-P 1700 4000
-F 0 "#PWR0106" H 1700 3850 50  0001 C CNN
-F 1 "VDD" H 1717 4173 50  0000 C CNN
-F 2 "" H 1700 4000 50  0001 C CNN
-F 3 "" H 1700 4000 50  0001 C CNN
-	1    1700 4000
 	1    0    0    -1
 $EndComp
@@
 Text Label 10350 4150 0    50   ~ 0
 PA6-Therm
+$Comp
+L power:+3.3V #PWR?
+U 1 1 5C4929D3
+P 1700 4000
+F 0 "#PWR?" H 1700 3850 50  0001 C CNN
+F 1 "+3.3V" H 1715 4173 50  0000 C CNN
+F 2 "" H 1700 4000 50  0001 C CNN
+F 3 "" H 1700 4000 50  0001 C CNN
+	1    1700 4000
+	1    0    0    -1
+$EndComp
 $EndSCHEMATC

Commit message: m
Parts:
- R3: renamed from R?; value 5 -> 10
- R4: renamed from R?; value 10 -> 6
- gave numbers to parts that had none: 28
Connections:
- net +3V3: no longer R3.2
- net +6V: now also R3.2
- net RX: no longer names the net of U6.22 (PD2)
- net TC: no longer names the net of U6.24 (PD4)
- net TC: no longer U6.25 (PD5)
- net TX: no longer names the net of U6.23 (PD3)
Other:
- note added: "RX"
- note added: "TC"
- note added: "TX\n"
- note added: "Voltage Divider (6 —> 2.25)"
- note removed: "Voltage Divider (3.3 —> 2.2)"

Commit message: m
Parts:
- added C?: C_Small, symbol Device:C_Small
- added R? (x2): R_Small, symbol Device:R_Small
- added U?: PCF8523T_1_118, digikey-footprints:SOIC-8_W3.9mm, symbol dk_Clock-Timing-Real-Time-Clocks:PCF8523T_1_118
- R3: value 10 -> 30k
- R4: value 6 -> 13k
Connections:
- net +3V3: now also R?.1, R?.1
- net GND: now also C?.1, U?.4 (VSS)
- new net: R?.2, U?.7 (~INT1~/CLKO)
- new net: C?.2, R?.2, U?.8 (VDD)
- new net I2C: U?.5 (SDA), U?.6 (SCL)
- no-connect marks 4 -> 7
Other:
- note added: "Real Time Clock"
- note added: "Voltage Divider (6 —> 2)"
- note removed: "Voltage Divider (6 —> 2.25)"
- moved on the sheet: C10, U5
