File: Electrical Design/PCB/PCB.kicad_pcb (KiCad board)
At the start: 2 copper layers, 50 x 150 mm, 59 parts, among them J1 PDI Interface, J2 10118193-0001LF, M1 Camera_Servo, M2 Release_Servo, Q1 LED_MOS, Q2 CAMERA_MOS, Q3 RELEASE_MOS, Q4 BUZZER_MOS, U1 6V-->5V, U10 Adafruit_Cam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

Commit message: m
Parts:
- J1: value PDI Interface -> Conn_02x03_Odd_Even
- U1: value 6V-->5V -> ADP3338AKCZ-5-R7
- U3: value 6V-->3.3V -> ADP3338AKCZ-3.3-R7
Connections:
- U7 pad 5: /GPS_TX -> /GPS_MISO
- U7 pad 6: /GPS_RX -> /GPS_MOSI
Changed lines of the file:
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@@
-(kicad_pcb (version 20171130) (host pcbnew 5.0.2-bee76a0~70~ubuntu18.04.1)
+(kicad_pcb (version 20171130) (host pcbnew "(5.0.1-3-g963ef8bb5)")
   (general
     (thickness 1.6)
@@
     (zones 0)
     (modules 59)
-    (nets 96)
+    (nets 94)
   )
   (page A4)
@@
   (net 73 "Net-(U7-Pad3)")
   (net 74 "Net-(U7-Pad4)")
-  (net 75 /GPS_TX)
-  (net 76 /GPS_RX)
-  (net 77 "Net-(U7-Pad9)")
-  (net 78 /OpenLog_MISO)
-  (net 79 /OpenLog_MOSI)
-  (net 80 /OpenLog_GRN)
-  (net 81 /PA5-Hall_Effect)
-  (net 82 "Net-(U9-Pad4)")
-  (net 83 "Net-(U9-Pad5)")
-  (net 84 "Net-(U9-Pad6)")
-  (net 85 "Net-(U9-Pad7)")
-  (net 86 /GPS_MISO)
-  (net 87 /GPS_MOSI)
-  (net 88 "Net-(U9-Pad24)")
-  (net 89 "Net-(U9-Pad25)")
-  (net 90 "Net-(U9-Pad26)")
-  (net 91 "Net-(U9-Pad27)")
-  (net 92 "Net-(U9-Pad36)")
-  (net 93 "Net-(U9-Pad37)")
-  (net 94 "Net-(U9-Pad44)")
-  (net 95 /CAMERA_DATA)
+  (net 75 "Net-(U7-Pad9)")
+  (net 76 /OpenLog_MISO)
+  (net 77 /OpenLog_MOSI)
+  (net 78 /OpenLog_GRN)
+  (net 79 /PA5-Hall_Effect)
+  (net 80 "Net-(U9-Pad4)")
+  (net 81 "Net-(U9-Pad5)")
+  (net 82 "Net-(U9-Pad6)")
+  (net 83 "Net-(U9-Pad7)")
+  (net 84 /GPS_MISO)
+  (net 85 /GPS_MOSI)
+  (net 86 "Net-(U9-Pad24)")
+  (net 87 "Net-(U9-Pad25)")
+  (net 88 "Net-(U9-Pad26)")
+  (net 89 "Net-(U9-Pad27)")
+  (net 90 "Net-(U9-Pad36)")
+  (net 91 "Net-(U9-Pad37)")
+  (net 92 "Net-(U9-Pad44)")
+  (net 93 /CAMERA_DATA)
   (net_class Default "This is the default net class."
     (clearance 0.1524)
@@
     (add_net /GPS_MISO)
     (add_net /GPS_MOSI)
-    (add_net /GPS_RX)
-    (add_net /GPS_TX)
     (add_net /HOST_INTN)
     (add_net /LED_MOS)
@@
       (effects (font (size 0.6096 0.6096) (thickness 0.127)))
     )
-    (fp_text value "PDI Interface" (at 0 2.286 270) (layer F.SilkS)
+    (fp_text value Conn_02x03_Odd_Even (at 0 2.286 270) (layer F.SilkS)
       (effects (font (size 0.6096 0.6096) (thickness 0.127)))
     )
@@
       (net 1 GND) (solder_mask_margin 0.1016))
     (pad 3 thru_hole circle (at 5.08 0 90) (size 1.8796 1.8796) (drill 1.016) (layers *.Cu *.Mask)
-      (net 95 /CAMERA_DATA) (solder_mask_margin 0.1016))
+      (net 93 /CAMERA_DATA) (solder_mask_margin 0.1016))
   )
   (module Capacitor_SMD:C_0805_2012Metric_Pad1.15x1.40mm_HandSolder (layer F.Cu)
@@
       (effects (font (size 1.64061 1.64061) (thickness 0.05)))
     )
-    (fp_text value 6V-->5V (at -0.5084 4.8298 90) (layer F.SilkS)
+    (fp_text value ADP3338AKCZ-5-R7 (at -0.5084 4.8298 90) (layer F.SilkS)
       (effects (font (size 1.64129 1.64129) (thickness 0.05)))
     )
@@
       (effects (font (size 1.64087 1.64087) (thickness 0.05)))
     )
-    (fp_text value 6V-->3.3V (at -0.508485 4.83074 90) (layer F.SilkS)
+    (fp_text value ADP3338AKCZ-3.3-R7 (at -0.508485 4.83074 90) (layer F.SilkS)
       (effects (font (size 1.64161 1.64161) (thickness 0.05)))
     )
@@
       (net 74 "Net-(U7-Pad4)") (solder_mask_margin 0.1016))
     (pad 5 thru_hole circle (at 10.16 0 90) (size 1.8796 1.8796) (drill 1.016) (layers *.Cu *.Mask)
-      (net 75 /GPS_TX) (solder_mask_margin 0.1016))
+      (net 84 /GPS_MISO) (solder_mask_margin 0.1016))
     (pad 6 thru_hole circle (at 12.7 0 90) (size 1.8796 1.8796) (drill 1.016) (layers *.Cu *.Mask)
-      (net 76 /GPS_RX) (solder_mask_margin 0.1016))
+      (net 85 /GPS_MOSI) (solder_mask_margin 0.1016))
     (pad 7 thru_hole circle (at 15.24 0 90) (size 1.8796 1.8796) (drill 1.016) (layers *.Cu *.Mask)
       (net 1 GND) (solder_mask_margin 0.1016))
@@
       (net 3 +3V3) (solder_mask_margin 0.1016))
     (pad 9 thru_hole circle (at 20.32 0 90) (size 1.8796 1.8796) (drill 1.016) (layers *.Cu *.Mask)
-      (net 77 "Net-(U7-Pad9)") (solder_mask_margin 0.1016))
+      (net 75 "Net-(U7-Pad9)") (solder_mask_margin 0.1016))
   )
   (module Connectors:1X06 (layer F.Cu)
@@
       (net 3 +3V3) (solder_mask_margin 0.1016))
     (pad 4 thru_hole circle (at 7.62 0 90) (size 1.8796 1.8796) (drill 1.016) (layers *.Cu *.Mask)
-      (net 78 /OpenLog_MISO) (solder_mask_margin 0.1016))
+      (net 76 /OpenLog_MISO) (solder_mask_margin 0.1016))
     (pad 5 thru_hole circle (at 10.16 0 90) (size 1.8796 1.8796) (drill 1.016) (layers *.Cu *.Mask)
-      (net 79 /OpenLog_MOSI) (solder_mask_margin 0.1016))
+      (net 77 /OpenLog_MOSI) (solder_mask_margin 0.1016))
     (pad 6 thru_hole circle (at 12.7 0 90) (size 1.8796 1.8796) (drill 1.016) (layers *.Cu *.Mask)
-      (net 80 /OpenLog_GRN) (solder_mask_margin 0.1016))
+      (net 78 /OpenLog_GRN) (solder_mask_margin 0.1016))
   )
   (module Package_QFP:TQFP-44_10x10mm_P0.8mm (layer F.Cu)
@@
     (fp_line (start -5.175 -4.6) (end -6.45 -4.6) (layer F.SilkS) (width 0.15))
     (pad 1 smd rect (at -5.7 -4 180) (size 1.5 0.55) (layers F.Cu F.Paste F.Mask)
-      (net 81 /PA5-Hall_Effect))
+      (net 79 /PA5-Hall_Effect))
     (pad 2 smd rect (at -5.7 -3.2 180) (size 1.5 0.55) (layers F.Cu F.Paste F.Mask)
       (net 47 /PA6-Therm))
@@
       (net 48 /PA7-Voltage))
     (pad 4 smd rect (at -5.7 -1.6 180) (size 1.5 0.55) (layers F.Cu F.Paste F.Mask)
-      (net 82 "Net-(U9-Pad4)"))
+      (net 80 "Net-(U9-Pad4)"))
     (pad 5 smd rect (at -5.7 -0.8 180) (size 1.5 0.55) (layers F.Cu F.Paste F.Mask)
-      (net 83 "Net-(U9-Pad5)"))
+      (net 81 "Net-(U9-Pad5)"))
     (pad 6 smd rect (at -5.7 0 180) (size 1.5 0.55) (layers F.Cu F.Paste F.Mask)
-      (net 84 "Net-(U9-Pad6)"))
+      (net 82 "Net-(U9-Pad6)"))
     (pad 7 smd rect (at -5.7 0.8 180) (size 1.5 0.55) (layers F.Cu F.Paste F.Mask)
-      (net 85 "Net-(U9-Pad7)"))
+      (net 83 "Net-(U9-Pad7)"))
     (pad 8 smd rect (at -5.7 1.6 180) (size 1.5 0.55) (layers F.Cu F.Paste F.Mask)
       (net 1 GND))
@@
       (net 50 /LED_MOS))
     (pad 21 smd rect (at 3.2 5.7 270) (size 1.5 0.55) (layers F.Cu F.Paste F.Mask)
-      (net 80 /OpenLog_GRN))
+      (net 78 /OpenLog_GRN))
     (pad 22 smd rect (at 4 5.7 270) (size 1.5 0.55) (layers F.Cu F.Paste F.Mask)
-      (net 86 /GPS_MISO))
+      (net 84 /GPS_MISO))
     (pad 23 smd rect (at 5.7 4 180) (size 1.5 0.55) (layers F.Cu F.Paste F.Mask)
-      (net 87 /GPS_MOSI))
+      (net 85 /GPS_MOSI))
     (pad 24 smd rect (at 5.7 3.2 180) (size 1.5 0.55) (layers F.Cu F.Paste F.Mask)
-      (net 88 "Net-(U9-Pad24)"))
+      (net 86 "Net-(U9-Pad24)"))
     (pad 25 smd rect (at 5.7 2.4 180) (size 1.5 0.55) (layers F.Cu F.Paste F.Mask)
-      (net 89 "Net-(U9-Pad25)"))
+      (net 87 "Net-(U9-Pad25)"))
     (pad 26 smd rect (at 5.7 1.6 180) (size 1.5 0.55) (layers F.Cu F.Paste F.Mask)
-      (net 90 "Net-(U9-Pad26)"))
+      (net 88 "Net-(U9-Pad26)"))
     (pad 27 smd rect (at 5.7 0.8 180) (size 1.5 0.55) (layers F.Cu F.Paste F.Mask)
-      (net 91 "Net-(U9-Pad27)"))
+      (net 89 "Net-(U9-Pad27)"))
     (pad 28 smd rect (at 5.7 0 180) (size 1.5 0.55) (layers F.Cu F.Paste F.Mask)
       (net 19 /Camera_Servo))
@@
       (net 7 /MCU_VCC))
     (pad 32 smd rect (at 5.7 -3.2 180) (size 1.5 0.55) (layers F.Cu F.Paste F.Mask)
-      (net 78 /OpenLog_MISO))
+      (net 76 /OpenLog_MISO))
     (pad 33 smd rect (at 5.7 -4 180) (size 1.5 0.55) (layers F.Cu F.Paste F.Mask)
-      (net 79 /OpenLog_MOSI))
+      (net 77 /OpenLog_MOSI))
     (pad 34 smd rect (at 4 -5.7 270) (size 1.5 0.55) (layers F.Cu F.Paste F.Mask)
       (net 11 /PDI_DATA))
@@
       (net 14 /PDI_CLK))
     (pad 36 smd rect (at 2.4 -5.7 270) (size 1.5 0.55) (layers F.Cu F.Paste F.Mask)
-      (net 92 "Net-(U9-Pad36)"))
+      (net 90 "Net-(U9-Pad36)"))
     (pad 37 smd rect (at 1.6 -5.7 270) (size 1.5 0.55) (layers F.Cu F.Paste F.Mask)
-      (net 93 "Net-(U9-Pad37)"))
+      (net 91 "Net-(U9-Pad37)"))
     (pad 38 smd rect (at 0.8 -5.7 270) (size 1.5 0.55) (layers F.Cu F.Paste F.Mask)
       (net 1 GND))
@@
       (net 51 /CAMERA_MOS))
     (pad 43 smd rect (at -3.2 -5.7 270) (size 1.5 0.55) (layers F.Cu F.Paste F.Mask)
-      (net 95 /CAMERA_DATA))
+      (net 93 /CAMERA_DATA))
     (pad 44 smd rect (at -4 -5.7 270) (size 1.5 0.55) (layers F.Cu F.Paste F.Mask)
-      (net 94 "Net-(U9-Pad44)"))
+      (net 92 "Net-(U9-Pad44)"))
     (model ${KISYS3DMOD}/Package_QFP.3dshapes/TQFP-44_10x10mm_P0.8mm.wrl
       (at (xyz 0 0 0))

Commit message: Progress baby
Routing:
- net +3V3: track 219.3 -> 420.4 mm
- net /LED_MOS: track 0.00 -> 104.7 mm, vias 0 -> 2
- net /~SS_5607: track 2.40 -> 98.2 mm, vias 0 -> 2
- net /Camera_Servo: track 0.00 -> 79.2 mm, vias 0 -> 2
- net /CAMERA_DATA: track 0.00 -> 78.3 mm, vias 0 -> 6
- net /CAMERA_MOS: track 0.00 -> 74.6 mm, vias 0 -> 6
- net /GPS_MOSI: track 0.00 -> 70.2 mm, vias 0 -> 2
- net /GPS_MISO: track 0.00 -> 68.4 mm, vias 0 -> 2
- net /PDI_CLK: track 0.00 -> 60.4 mm, vias 0 -> 6
- net /MISO: track 28.2 -> 87.9 mm, vias 3 -> 10
- net /SCLK: track 0.00 -> 52.6 mm, vias 0 -> 5
- net /~SS_BNO080: track 0.00 -> 48.9 mm, vias 0 -> 3
- net /SCL: track 0.00 -> 47.1 mm, vias 0 -> 8
- net /MOSI: track 16.8 -> 60.6 mm, vias 1 -> 9
- net /~SS_XBEE: track 0.00 -> 43.4 mm, vias 0 -> 8
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
Commit message: a
Connections:
- U6 pad 3: /PA5-Hall_effect -> /PA5-Hall_Effect
