File: Electrical Design/PCB/PCB.kicad_pcb (KiCad board)
At the start: 2 copper layers, 50 x 150 mm, 59 parts, among them J1 Conn_02x03_Odd_Even, J2 10118193-0001LF, M1 Camera_Servo, M2 Release_Servo, Q1 LED_MOS, Q2 CAMERA_MOS, Q3 RELEASE_MOS, Q4 BUZZER_MOS, U1 ADP3338AKCZ-5-R7, U10 Adafruit_Cam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

Commit message: I think its done, but holy shit its bad
Routing:
- net /Release_Servo: track 0.00 -> 226.5 mm, vias 0 -> 4
- net /PA5-Hall_Effect: track 0.00 -> 198.7 mm, vias 0 -> 4
- net +5V: track 33.4 -> 176.6 mm
- net /OpenLog_MISO: track 0.00 -> 126.5 mm, vias 0 -> 6
- net /BUZZER_MOS: track 0.00 -> 125.1 mm, vias 0 -> 13
- net /OpenLog_GRN: track 0.00 -> 91.4 mm, vias 0 -> 4
- net /OpenLog_MOSI: track 4.27 -> 93.0 mm, vias 2 -> 7
- net /RELEASE_MOS: track 0.00 -> 73.0 mm, vias 0 -> 4
- net GND: track 0.00 -> 51.4 mm, vias 0 -> 9
- net +6V: track 223.2 -> 258.4 mm, vias 2 -> 4
- net (no net): track 0.00 -> 12.5 mm, vias 0 -> 2
- net Net-(J2-PadSH): track 0.00 -> 12.4 mm
- net Net-(D5-PadA): track 0.00 -> 9.17 mm
- net +3V3: track 420.4 -> 426.8 mm
- net Net-(Q3-Pad3): track 0.00 -> 5.25 mm
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- added copper zone on B.Cu, net GND
- added copper zone on F.Cu, net GND

Commit message: Its fuckin done
Routing:
- net GND: track 51.4 -> 321.5 mm, vias 9 -> 37
- net (no net): track 12.5 -> 0.00 mm, vias 2 -> 0
- net /BUZZER_MOS: track 125.1 -> 122.1 mm
- net /MCU_VCC: track 80.1 -> 81.2 mm
- net /~SS_5607: track 98.2 -> 98.8 mm

Commit message: update pcb
Parts:
- removed R13: 10k, Resistor_SMD:R_0805_2012Metric_Pad1.15x1.40mm_HandSolder
- removed R14: 10K, Resistor_SMD:R_0805_2012Metric_Pad1.15x1.40mm_HandSolder
- added C17: 100nF, Capacitor_SMD:C_0805_2012Metric_Pad1.15x1.40mm_HandSolder, F.Cu at (46.3, 15.6)
- added C18: 100nF, Capacitor_SMD:C_0805_2012Metric_Pad1.15x1.40mm_HandSolder, F.Cu at (46.3, 13.7)
- R12: value 10k -> 10K
- U1: value ADP3338AKCZ-5-R7 -> Adafruit_Cam; footprint ADP3338AKCZ-5-R7:SOT230P700X180-4N -> Connectors:MOLEX-1X3
- U10: value Adafruit_Cam -> ATxmega128A4U-AU; footprint Connectors:MOLEX-1X3 -> Package_QFP:TQFP-44_10x10mm_P0.8mm
- U2: value BNO080 -> ADP3338AKCZ-5-R7; footprint BNO080:LGA-28 -> ADP3338AKCZ-5-R7:SOT230P700X180-4N
- U3: value ADP3338AKCZ-3.3-R7 -> BNO080; footprint ADP3338AKCZ-3.3RL7:SOT230P700X180-4N -> BNO080:LGA-28
- U4: value PCF8523T_1_118 -> ADP3338AKCZ-3.3-R7; footprint digikey-footprints:SOIC-8_W3.9mm -> ADP3338AKCZ-3.3RL7:SOT230P700X180-4N
- U5: value MS560702BA03-50 -> PCF8523T_1_118; footprint MS560702BA03-50:SON125P300X500X100-8N -> digikey-footprints:SOIC-8_W3.9mm
- U6: value SS495A -> MS560702BA03-50; footprint Connector_PinHeader_2.00mm:PinHeader_1x03_P2.00mm_Horizontal -> MS560702BA03-50:SON125P300X500X100-8N
- U7: value Adafruit_746 -> SS495A; footprint Connectors:1X09 -> Connector_PinHeader_2.00mm:PinHeader_1x03_P2.00mm_Horizontal
- U9: value ATxmega128A4U-AU -> Adafruit_746; footprint Package_QFP:TQFP-44_10x10mm_P0.8mm -> Connectors:1X09
Connections:
- C16 pad 1: GND -> /MCU_VCC
- C16 pad 2: /MCU_AVCC -> GND
- Q2 pad 3: Net-(Q2-Pad3) -> Net-(M1-Pad3)
- Q3 pad 3: Net-(Q3-Pad3) -> Net-(M2-Pad3)
- R10 pad 1: Net-(Q2-Pad3) -> +3V3
- R10 pad 2: Net-(M1-Pad3) -> /SCL
- R11 pad 1: Net-(Q3-Pad3) -> +3V3
- R11 pad 2: Net-(M2-Pad3) -> /SDA
- R12 pad 1: +3V3 -> /BUZZER_MOS
- R12 pad 2: /SCL -> Net-(Q4-Pad1)
- U1 pad 1: GND -> +5V
- U1 pad 2: +5V -> GND
- U1 pad 3: +6V -> /CAMERA_DATA
- U10 pad 1: +5V -> /PA5-Hall_Effect
- U10 pad 2: GND -> /PA6-Therm
- U10 pad 3: /CAMERA_DATA -> /PA7-Voltage
- U2 pad 1: (no net) -> GND
- U2 pad 2: GND -> +5V
- U2 pad 3: +3V3 -> +6V
- U2 pad 4: /BNO_BOOTN -> +5V
- U3 pad 1: GND -> (no net)
- U3 pad 2: +3V3 -> GND
- U3 pad 3: +6V -> +3V3
- U3 pad 4: +3V3 -> /BNO_BOOTN
- U4 pad 1: Net-(U4-Pad1) -> GND
- U4 pad 2: Net-(U4-Pad2) -> +3V3
- U4 pad 3: Net-(U4-Pad3) -> +6V
- U4 pad 4: GND -> +3V3
- U5 pad 1: +3V3 -> Net-(U5-Pad1)
- U5 pad 2: GND -> Net-(U5-Pad2)
- U5 pad 3: GND -> Net-(U5-Pad3)
- U5 pad 4: /~SS_5607 -> GND
- U5 pad 5: /~SS_5607 -> /SDA
- U5 pad 6: /MISO -> /SCL
- U5 pad 7: /MOSI -> Net-(R6-Pad2)
- U5 pad 8: /SCLK -> Net-(C8-Pad2)
- U6 pad 1: +5V -> +3V3
- U6 pad 3: /PA5-Hall_Effect -> GND
- U7 pad 1: Net-(U7-Pad1) -> +5V
- U7 pad 2: Net-(U7-Pad2) -> GND
- U7 pad 3: Net-(U7-Pad3) -> /PA5-Hall_Effect
- U9 pad 1: /PA5-Hall_Effect -> Net-(U9-Pad1)
- U9 pad 2: /PA6-Therm -> Net-(U9-Pad2)
- U9 pad 3: /PA7-Voltage -> Net-(U9-Pad3)
- U9 pad 5: Net-(U9-Pad5) -> /GPS_MISO
- U9 pad 6: Net-(U9-Pad6) -> /GPS_MOSI
- U9 pad 7: Net-(U9-Pad7) -> GND
- U9 pad 8: GND -> +3V3
- U9 pad 9: /MCU_VCC -> Net-(U9-Pad9)
Routing:
- net Net-(U5-Pad2): track 0.00 -> 98.8 mm, vias 0 -> 2
- net /~SS_5607: track 98.8 -> 0.00 mm, vias 2 -> 0
- net /CAMERA_DATA: track 78.3 -> 0.00 mm, vias 6 -> 0
- net /Camera_Servo: track 79.2 -> 157.4 mm, vias 2 -> 8
