File: Electrical Design/PCBV2/PCB.kicad_pcb (KiCad board)
At the start: 2 copper layers, 65 x 80 mm, 62 parts, among them J1 PDI_Interface, J2 10118193-0001LF, M1 Finn_servo, M2 Release_Servo, Q1 LED_MOS, Q2 FINN_MOS, Q3 RELEASE_MOS, Q4 BUZZER_MOS, Q5 CAMERA_MOS, U1 Adafruit_Cam, U2 BNO080, U3 6->3V3, U4 RTC, U5 MS560702BA03-50, U6 SS49E, U7 Openlog, U8 Adafruit_746, U9 ATxmega128A4U-AU

Commit message: Final changes
Routing:
- net +3V3: track 323.3 -> 327.1 mm
- net GND: track 179.7 -> 182.6 mm, vias 21 -> 38
- net (no net): track 0.72 -> 3.03 mm, vias 0 -> 1
Other:
- board size 65 x 80 mm -> 66 x 81 mm
Changed lines of the file:
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@@
     (thickness 1.6)
     (drawings 6)
-    (tracks 842)
+    (tracks 870)
     (zones 0)
     (modules 62)
@@
   )
   (layers
-    (0 F.Cu signal hide)
-    (31 B.Cu signal hide)
+    (0 F.Cu signal)
+    (31 B.Cu signal)
     (32 B.Adhes user)
     (33 F.Adhes user)
@@
       (effects (font (size 1 1) (thickness 0.15)) (justify mirror))
     )
-    (fp_text value CAMERA_MOS (at 0.025 -3.25 270) (layer B.Fab)
+    (fp_text value CAMERA_MOS (at -1.744 -3.25 270) (layer B.Fab)
       (effects (font (size 1 1) (thickness 0.15)) (justify mirror))
     )
@@
       (effects (font (size 1 1) (thickness 0.15)) (justify mirror))
     )
-    (fp_text value FINN_MOS (at 0.025 -3.25 270) (layer B.Fab)
+    (fp_text value FINN_MOS (at -0.22 -3.25 270) (layer B.Fab)
       (effects (font (size 1 1) (thickness 0.15)) (justify mirror))
     )
@@
     (effects (font (size 1.5 1.5) (thickness 0.3)))
   )
-  (gr_line (start 104.242 48.194) (end 169.242 48.194) (layer Edge.Cuts) (width 0.2))
-  (gr_line (start 169.242 48.194) (end 169.242 128.194) (layer Edge.Cuts) (width 0.2))
-  (gr_line (start 104.242 128.194) (end 169.242 128.194) (layer Edge.Cuts) (width 0.2))
-  (gr_line (start 104.242 48.194) (end 104.242 128.194) (layer Edge.Cuts) (width 0.2))
+  (gr_line (start 103.742 47.694) (end 169.742 47.694) (layer Edge.Cuts) (width 0.2))
+  (gr_line (start 169.742 47.694) (end 169.742 128.694) (layer Edge.Cuts) (width 0.2))
+  (gr_line (start 103.742 128.694) (end 169.742 128.694) (layer Edge.Cuts) (width 0.2))
+  (gr_line (start 103.742 47.694) (end 103.742 128.694) (layer Edge.Cuts) (width 0.2))
   (segment (start 121.711601 49.230399) (end 121.412 49.53) (width 0.2032) (layer F.Cu) (net 0))
   (segment (start 116.332 50.9905) (end 116.332 51.282599) (width 0.2032) (layer F.Cu) (net 0))
+  (via (at 145.288 101.854) (size 0.762) (drill 0.381) (layers F.Cu B.Cu) (net 0))
+  (via (at 123.698 73.66) (size 0.762) (drill 0.381) (layers F.Cu B.Cu) (net 1))
+  (via (at 122.428 68.834) (size 0.762) (drill 0.381) (layers F.Cu B.Cu) (net 1))
+  (via (at 122.428 64.77) (size 0.762) (drill 0.381) (layers F.Cu B.Cu) (net 1))
+  (via (at 144.272 66.802) (size 0.762) (drill 0.381) (layers F.Cu B.Cu) (net 1))
+  (via (at 158.75 71.628) (size 0.762) (drill 0.381) (layers F.Cu B.Cu) (net 1))
+  (via (at 159.004 82.55) (size 0.762) (drill 0.381) (layers F.Cu B.Cu) (net 1))
+  (via (at 120.142 118.364) (size 0.762) (drill 0.381) (layers F.Cu B.Cu) (net 1))
+  (via (at 164.084 115.316) (size 0.762) (drill 0.381) (layers F.Cu B.Cu) (net 1))
+  (via (at 139.7 114.808) (size 0.762) (drill 0.381) (layers F.Cu B.Cu) (net 1))
+  (via (at 107.696 108.712) (size 0.762) (drill 0.381) (layers F.Cu B.Cu) (net 1))
+  (via (at 106.934 114.808) (size 0.762) (drill 0.381) (layers F.Cu B.Cu) (net 1))
+  (via (at 142.494 57.658) (size 0.762) (drill 0.381) (layers F.Cu B.Cu) (net 1))
+  (via (at 139.446 57.658) (size 0.762) (drill 0.381) (layers F.Cu B.Cu) (net 1))
+  (via (at 132.842 117.602) (size 0.762) (drill 0.381) (layers F.Cu B.Cu) (net 1))
+  (via (at 161.544 121.666) (size 0.762) (drill 0.381) (layers F.Cu B.Cu) (net 1))
+  (via (at 106.426 87.122) (size 0.762) (drill 0.381) (layers F.Cu B.Cu) (net 1))
+  (via (at 159.004 88.9) (size 0.762) (drill 0.381) (layers F.Cu B.Cu) (net 1))
+  (segment (start 144.907001 102.234999) (end 144.907001 104.013001) (width 0.2032) (layer B.Cu) (net 0))
+  (segment (start 145.288 101.854) (end 144.907001 102.234999) (width 0.2032) (layer B.Cu) (net 0))
+  (segment (start 139.7 114.808) (end 139.7 112.522) (width 0.2032) (layer B.Cu) (net 1))
+  (segment (start 132.842 117.602) (end 132.842 117.063185) (width 0.2032) (layer B.Cu) (net 1))
   (segment (start 107.188 65.980923) (end 107.188 64.77) (width 0.2032) (layer F.Cu) (net 1))
   (segment (start 107.188 67.31) (end 107.188 65.980923) (width 0.2032) (layer F.Cu) (net 1))
@@
   (segment (start 120.336923 127.508) (end 117.602 124.773077) (width 0.635) (layer F.Cu) (net 2))
   (segment (start 150.368 127.508) (end 120.336923 127.508) (width 0.635) (layer F.Cu) (net 2))
-  (segment (start 120.336923 127.508) (end 114.554 127.508) (width 0.635) (layer F.Cu) (net 2))
-  (segment (start 114.554 127.508) (end 110.236 123.19) (width 0.635) (layer F.Cu) (net 2))
-  (segment (start 110.236 123.19) (end 110.236 97.282) (width 0.635) (layer F.Cu) (net 2))
   (segment (start 110.236 97.282) (end 112.776 94.742) (width 0.635) (layer F.Cu) (net 2))
   (via (at 121.666 94.742) (size 0.762) (drill 0.381) (layers F.Cu B.Cu) (net 2))
@@
   (segment (start 113.792 52.324) (end 113.792 50.7492) (width 0.635) (layer F.Cu) (net 2))
   (segment (start 113.792 50.7492) (end 114.5032 50.038) (width 0.635) (layer F.Cu) (net 2))
+  (segment (start 110.236 122.428) (end 110.236 97.282) (width 0.635) (layer F.Cu) (net 2))
+  (segment (start 120.336923 127.508) (end 115.316 127.508) (width 0.635) (layer F.Cu) (net 2))
+  (segment (start 115.316 127.508) (end 110.236 122.428) (width 0.635) (layer F.Cu) (net 2))
   (segment (start 158.0134 118.364) (end 158.0134 117.9957) (width 0.254) (layer B.Cu) (net 3))
   (segment (start 167.563799 62.153799) (end 166.624 61.214) (width 0.254) (layer F.Cu) (net 3))
@@
   (segment (start 168.402 62.992) (end 168.402 57.912) (width 0.254) (layer F.Cu) (net 3))
   (segment (start 146.558 48.768) (end 146.05 49.276) (width 0.254) (layer F.Cu) (net 3))
-  (segment (start 168.402 57.912) (end 159.258 48.768) (width 0.254) (layer F.Cu) (net 3))
   (segment (start 146.05 50.8) (end 146.05 52.832) (width 0.254) (layer F.Cu) (net 3))
   (segment (start 147.796 50.8) (end 148.16 50.436) (width 0.254) (layer F.Cu) (net 3))
@@
   (segment (start 122.682 92.456) (end 122.682 93.472) (width 0.2032) (layer F.Cu) (net 3))
   (segment (start 122.428 92.202) (end 122.682 92.456) (width 0.2032) (layer F.Cu) (net 3))
+  (segment (start 168.402 55.626) (end 168.402 57.912) (width 0.2032) (layer F.Cu) (net 3))
+  (segment (start 161.29 48.768) (end 162.306 49.784) (width 0.2032) (layer F.Cu) (net 3))
+  (segment (start 162.306 54.102) (end 163.576 55.372) (width 0.2032) (layer F.Cu) (net 3))
+  (segment (start 162.306 49.784) (end 162.306 54.102) (width 0.2032) (layer F.Cu) (net 3))
+  (segment (start 159.258 48.768) (end 161.29 48.768) (width 0.2032) (layer F.Cu) (net 3))
+  (segment (start 168.148 55.372) (end 168.402 55.626) (width 0.2032) (layer F.Cu) (net 3))
+  (segment (start 163.576 55.372) (end 168.148 55.372) (width 0.2032) (layer F.Cu) (net 3))
   (segment (start 138.557 97.409) (end 138.557 95.885) (width 0.254) (layer F.Cu) (net 4))
   (segment (start 138.342 95.67) (end 138.342 93.894) (width 0.254) (layer F.Cu) (net 4))
