File: Electrical Design/PCBV2/PCB.kicad_pcb (KiCad board)
At the start: 2 copper layers, 66 x 81 mm, 62 parts, among them J1 PDI_Interface, J2 10118193-0001LF, M1 Finn_servo, M2 Release_Servo, Q1 LED_MOS, Q2 FINN_MOS, Q3 RELEASE_MOS, Q4 BUZZER_MOS, Q5 CAMERA_MOS, U1 Adafruit_Cam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

Commit message: bugfixes
Parts:
- added M3: Finn_Servo_Two, Connectors:MOLEX-1X3_LOCK, F.Cu at (126.7, 123.7)
- added R14: 10K, Resistor_SMD:R_0805_2012Metric_Pad1.15x1.40mm_HandSolder, F.Cu at (163.1, 109.5)
- added R15: 10K, Resistor_SMD:R_0805_2012Metric_Pad1.15x1.40mm_HandSolder, F.Cu at (161.8, 101.9)
- added R16: 10K, Resistor_SMD:R_0805_2012Metric_Pad1.15x1.40mm_HandSolder, F.Cu at (161.3, 105.7)
- M1: value Finn_servo -> Finn_Servo_One
- moved R13 5.60 mm to (130.8, 115.3), turned to 0 degrees
- moved Q5 4.32 mm to (130.8, 118.6)
- moved C11 4.32 mm to (153.4, 102.1)
- moved L1 4.32 mm to (153.4, 105.3)
- moved U1 4.32 mm to (135.9, 123.7)
- moved M1 2.54 mm to (117.6, 123.6)
- moved D2 1.81 mm to (167.3, 109.5)
- moved R9 1.43 mm to (159.8, 62.2), turned to 180 degrees
- moved G*** 1.08 mm to (116.1, 64.0)
- moved R12 0.13 mm to (123.6, 89.9), turned to 0 degrees
Connections:
- D1 pad 2: +6V -> Net-(D1-Pad2)
- D2 pad 2: +3V3 -> Net-(D2-Pad2)
- D4 pad 2: +6V -> Net-(D4-Pad2)
- M1 pad 1: /FINN_SERVO -> /FINN_SERVO_ONE
- Q1 pad 1: Net-(Q1-Pad1) -> /LED_MOS
- Q2 pad 1: Net-(Q2-Pad1) -> /FINN_MOS
- Q2 pad 2: GND -> Net-(Q2-Pad2)
- Q3 pad 1: Net-(Q3-Pad1) -> /RELEASE_MOS
- Q4 pad 1: Net-(Q4-Pad1) -> /BUZZER_MOS
- Q5 pad 1: Net-(Q5-Pad1) -> /CAMERA_DATA
- R12 pad 1: /BUZZER_MOS -> +6V
- R12 pad 2: Net-(Q4-Pad1) -> /BUZZER_MOS
- R13 pad 1: Net-(Q5-Pad1) -> /CAMERA_DATA
- R13 pad 2: /CAMERA_DATA -> +3V3
- R7 pad 1: /LED_MOS -> +6V
- R7 pad 2: Net-(Q1-Pad1) -> /LED_MOS
- R8 pad 2: Net-(Q2-Pad1) -> +6V
- R9 pad 2: Net-(Q3-Pad1) -> +6V
- U9 pad 26: Net-(U9-Pad26) -> /FINN_SERVO_ONE
- U9 pad 28: /Camera_Servo -> /FINN_SERVO_TWO
Routing:
- net /FINN_SERVO_ONE: track 0.00 -> 68.5 mm, vias 0 -> 3
- net /FINN_SERVO_TWO: track 0.00 -> 61.8 mm, vias 0 -> 3
- net +6V: track 243.7 -> 277.5 mm, vias 7 -> 9
- net Net-(M1-Pad3): track 4.06 -> 23.5 mm, vias 0 -> 3
- net GND: track 182.6 -> 171.3 mm
- net /BUZZER_MOS: track 18.5 -> 26.9 mm
- net /CAMERA_DATA: track 46.0 -> 54.0 mm
- net Net-(Q4-Pad1): track 5.43 -> 0.00 mm
- net /FINN_MOS: track 59.2 -> 64.5 mm
- net /RELEASE_MOS: track 48.3 -> 52.9 mm
- net /LED_MOS: track 26.8 -> 30.5 mm
- net +3V3: track 327.1 -> 330.6 mm, vias 3 -> 4
- net /MCU_VCC: track 67.3 -> 64.4 mm
- net (no net): track 3.03 -> 0.72 mm, vias 1 -> 3
- net Net-(D2-Pad2): track 0.00 -> 2.30 mm
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
Commit message: fix logo
Parts:
- moved G*** 37.5 mm to (140.5, 92.5)
