File: Electrical Design/PCBV2/PCB.sch (KiCad schematic (older format))
At the start: 59 parts, among them J1 Conn_02x03_Odd_Even, J2 10118193-0001LF, M1 Camera_Servo, M2 Release_Servo, Q1 LED_MOS, Q2 CAMERA_MOS, Q3 RELEASE_MOS, Q4 BUZZER_MOS, U1 Adafruit_Cam, U10 ATxmega128A4U-AU, U2 ADP3338AKCZ-5-R7, U3 BNO080, U4 ADP3338AKCZ-3.3-R7, U5 PCF8523T_1_118, U6 MS560702BA03-50, U7 SS495A, U8 Openlog, U9 Adafruit_746

Commit message: fix the libraries
Parts:
- U1: symbol Skyfire_Custom_Components:Adafruit_Cam -> PCB-rescue:Adafruit_Cam-Skyfire_Custom_Components
Changed lines of the file:
@@
 $EndComp
 $Comp
-L Skyfire_Custom_Components:Adafruit_Cam U1
+L PCB-rescue:Adafruit_Cam-Skyfire_Custom_Components U1
 U 1 1 5C5F2365
 P -1350 2200

Commit message: major revision progress
Parts:
- removed C13, C15: 10uF, Capacitor_THT:CP_Radial_D10.0mm_P5.00mm, symbol Device:CP1_Small
- removed C2, C3, C5: 0.1uF, Capacitor_THT:CP_Radial_D5.0mm_P2.00mm, symbol Device:CP1_Small
- removed C6: 1uF, Capacitor_SMD:C_0805_2012Metric_Pad1.15x1.40mm_HandSolder, symbol Device:C_Small
- removed U2: ADP3338AKCZ-5-R7, ADP3338AKCZ-5-R7:SOT230P700X180-4N, symbol PCB-rescue:ADP3338AKCZ-5-R7-ADP3338AKCZ-5-R7
- added C11, C13: 10uF, Capacitor_SMD:C_0805_2012Metric_Pad1.15x1.40mm_HandSolder, symbol Device:C_Small
- added C2, C4: 0.1uF, Capacitor_SMD:C_0805_2012Metric_Pad1.15x1.40mm_HandSolder, symbol Device:C_Small
- added H1, H2, H3, H4: MountingHole, MountingHole:MountingHole_3.2mm_M3, symbol Mechanical:MountingHole
- added Q5: CAMERA_MOS, digikey-footprints:SOT-23-3, symbol PCB-rescue:2N7002K-T1-E3-dk_Transistors-FETs-MOSFETs-Single
- added R13: 10K, Resistor_SMD:R_0805_2012Metric_Pad1.15x1.40mm_HandSolder, symbol Device:R_Small
- BT1: footprint Connectors:MOLEX-1X2 -> Connectors:MOLEX-1X2_LOCK
- C1: value 1uF -> 0.1uF
- J1: value Conn_02x03_Odd_Even -> PDI_Interface
- M1: value Camera_Servo -> Finn_servo; footprint Connector_PinHeader_2.54mm:PinHeader_1x03_P2.54mm_Horizontal -> Connectors:MOLEX-1X3_LOCK
- M2: footprint Connector_PinHeader_2.54mm:PinHeader_1x03_P2.54mm_Horizontal -> Connectors:MOLEX-1X3_LOCK
- Q2: value CAMERA_MOS -> FINN_MOS
- U1: footprint Connectors:MOLEX-1X3 -> Connectors:MOLEX-1X3_LOCK
- U3: renamed from U4; value ADP3338AKCZ-3.3-R7 -> 6->3V3
- U4: renamed from U5; value PCF8523T_1_118 -> RTC
- U6: renamed from U7; value SS495A -> SS49E; footprint Connector_PinHeader_2.00mm:PinHeader_1x03_P2.00mm_Horizontal -> Connectors:MOLEX-1X3_LOCK
- renumbered C12 to C10, C14 to C12, C16 to C14, C17 to C15, C18 to C16, C4 to C3, C7 to C5, C8 to C6, C9 to C7, C10 to C8, C11 to C9, U3 to U2, U6 to U5, U8 to U7, U9 to U8, U10 to U9
Connections:
- net +3V3: now also C1.1, U1.1 (Vin), C2.1
- net +5V: no longer C9.2, U1.1 (Vin), U6.1 (VCC)
- net +6V: now also C9.2, U6.1 (VCC); no longer C1.2
- net CAMERA_DATA: now also R13.2; no longer U1.3 (DATA)
- net Camera_Servo: no longer M1.1 (PWM)
- net GND: now also C1.2, C11.2, C13.1, C2.2, C4.2, Q5.2 (S); no longer C1.1
- net MCU_AVCC: now also C13.2
- net MCU_VCC: now also C11.1
- net at U2.9 (CAP): now also C4.1
- net CAMERA_MOS renamed FINN_MOS
- new net: Q5.3 (D), U1.3 (DATA)
- new net: Q5.1 (G), R13.1
- new net FINN_SERVO: M1.1 (PWM)
Other:
- note removed: "6V —> 5V Regulator"
- moved on the sheet: BT1

Commit message: bugfixes
Parts:
- removed D3: 5V Status, LED_SMD:LED_0603_1608Metric_Pad1.05x0.95mm_HandSolder, symbol Device:LED
- added M3: Finn_Servo_Two, Connectors:MOLEX-1X3_LOCK, symbol Motor:Motor_Servo
- added R14, R15, R16: 10K, Resistor_SMD:R_0805_2012Metric_Pad1.15x1.40mm_HandSolder, symbol Device:R_Small
- M1: value Finn_servo -> Finn_Servo_One
Connections:
- net FINN_SERVO is gone; now on net FINN_SERVO_ONE: M1.1 (PWM)
- net +3V3: now also R13.2, R14.1; no longer D2.2 (A)
- net +6V: now also R12.1, R7.1, R8.2, R9.2, M3.2 (+), R15.1, R16.1; no longer D1.2 (A), D4.2 (A)
- net BUZZER_MOS: now also Q4.1 (G), R12.2; no longer R12.1
- net CAMERA_DATA: now also Q5.1 (G), R13.1; no longer R13.2
- net FINN_MOS: now also Q2.1 (G)
- net GND: no longer Q2.2 (S)
- net LED_MOS: now also Q1.1 (G), R7.2; no longer R7.1
- net RELEASE_MOS: now also Q3.1 (G)
- net FINN_SERVO_ONE: now reaches U9.26 (PD6)
- net at M1.3 (-), Q2.3 (D): now also M3.3 (-)
- net Camera_Servo renamed FINN_SERVO_TWO
- net FINN_SERVO_TWO: now also M3.1 (PWM)
- new net: D2.2 (A), R14.2
- new net: D4.2 (A), R16.2
- new net: D1.2 (A), R15.2
Other:
- moved on the sheet: D2, D4, M1, Q2, R12, R13, R7, R8, R9
